Commit message: updated motion demo files

File: demos/motion_demo/src/hebi_description/urdf/robot.urdf (robot description, URDF)
Before this commit: robot arm_demo, 14 links, 13 joints
Joints:
- removed joint motor1/X5_4
- removed joint motor2/X5_4
- added joint motor1/X5_9: type continuous, parent motor1/INPUT_INTERFACE, child right_arm1/INPUT_INTERFACE, origin xyz=0 0 0.031 rpy=0 0 0, axis 0 0 1, limit effort=13.0 velocity=14
- added joint motor2/X5_9: type continuous, parent motor2/INPUT_INTERFACE, child right_arm2/INPUT_INTERFACE, origin xyz=0 0 0.031 rpy=0 0 0, axis 0 0 1, limit effort=13.0 velocity=14
