Commit message: updated moveit_ws with new urdfs and taskspace checker code.

File: moveit_ws/src/hebi_description/urdf/4dof_robot.urdf (robot description, URDF)
Before this commit: robot arm_demo, 16 links, 15 joints
Links:
- link right_arm2/INPUT_INTERFACE: mass 0.36468 -> 0.33968; geometry collision cylinder length=0.1438 radius=.016; collision mesh filename=package://hebi_description/meshes/A-2038-02.stl
- link sensor/INPUT_INTERFACE: mass 0.37436 -> 0.34936; geometry collision cylinder length=0.168 radius=.016; collision mesh filename=package://hebi_description/meshes/A-2038-02.stl
Joints:
- joint end_joint: origin xyz=0.2559 0 0.02 rpy=0 0 0 -> xyz=0.1934 0 0.02 rpy=0 0 0
- joint right_arm2/OUTPUT_JOINT: origin xyz=0.2317 -0.0165942524924 0.00883618415505 rpy=2.163 0 0 -> xyz=0.1692 -0.0165942524924 0.00883618415505 rpy=2.163 0 0

File: moveit_ws/src/hebi_description/urdf/4dof_robot.xacro (robot description, xacro)
@@ -148,9 +148,9 @@
   <xacro:x_tube_link name="right_arm1" child="motor2" extension="0.125" twist="1.3343"/>
   <xacro:x5 joint="motor2" child="right_arm2" model="X5_9"/>
-  <xacro:x_tube_link name="right_arm2" child="motor3" extension="0.2317" twist="2.1630"/>
+  <xacro:x_tube_link name="right_arm2" child="motor3" extension="0.1692" twist="2.1630"/>
   <xacro:x5 joint="motor3" child="right_arm3" model="X5_9"/>
   <xacro:x_tube_link name="right_arm3" child="motor4" extension="0.2048" twist="-3.7736" />
   <xacro:x5 joint="motor4" child="sensor" model="X5_4" />
-  <xacro:sensor_mac name="sensor" child="end_link" extension="0.2559"/>
+  <xacro:sensor_mac name="sensor" child="end_link" extension="0.1934"/>
    <!-- end link -->
   <link name="end_link/INPUT_INTERFACE">

File: moveit_ws/src/hebi_description/urdf/5dof_yaxismotor_robot.urdf (robot description, URDF)
Before this commit: robot arm_demo, 18 links, 17 joints
Links:
- link right_arm3/INPUT_INTERFACE: mass 0.322 -> 0.33836; geometry collision cylinder length=0.1405 radius=.016; collision mesh filename=package://hebi_description/meshes/A-2038-02.stl
Joints:
- joint right_arm3/OUTPUT_JOINT: origin xyz=0.125 -0.0187480333335 0.0130349984833 rpy=1.9265 0 0 -> xyz=0.1659 -0.0187480333335 0.0130349984833 rpy=1.9265 0 0

File: moveit_ws/src/hebi_description/urdf/5dof_yaxismotor_robot.xacro (robot description, xacro)
@@ -150,5 +150,5 @@
   <xacro:x_tube_link name="right_arm2" child="motor3" extension="0.125" twist="0.2365"/>
   <xacro:x5 joint="motor3" child="right_arm3" model="X5_9"/>
-  <xacro:x_tube_link name="right_arm3" child="motor4" extension="0.125" twist="1.9265"/>
+  <xacro:x_tube_link name="right_arm3" child="motor4" extension="0.1659" twist="1.9265"/>
   <xacro:x5 joint="motor4" child="right_arm4" model="X5_9"/>
   <xacro:x_tube_link name="right_arm4" child="motor5" extension="0.13315" twist="-3.7736" />

File: moveit_ws/src/hebi_description/urdf/5dof_zaxismotor_robot.urdf (robot description, URDF)
Before this commit: robot arm_demo, 18 links, 17 joints
Links:
- link right_arm3/INPUT_INTERFACE: mass 0.322 -> 0.33836; geometry collision cylinder length=0.1405 radius=.016; collision mesh filename=package://hebi_description/meshes/A-2038-02.stl
Joints:
- joint right_arm3/OUTPUT_JOINT: origin xyz=0.125 0.00696507038204 0.00125199225055 rpy=3.4973 0 0 -> xyz=0.1659 0.00696507038204 0.00125199225055 rpy=3.4973 0 0

File: moveit_ws/src/hebi_description/urdf/5dof_zaxismotor_robot.xacro (robot description, xacro)
@@ -150,5 +150,5 @@
   <xacro:x_tube_link name="right_arm2" child="motor3" extension="0.125" twist="-1.3343"/>
   <xacro:x5 joint="motor3" child="right_arm3" model="X5_9"/>
-  <xacro:x_tube_link name="right_arm3" child="motor4" extension="0.125" twist="3.4973"/>
+  <xacro:x_tube_link name="right_arm3" child="motor4" extension="0.1659" twist="3.4973"/>
   <xacro:x5 joint="motor4" child="right_arm4" model="X5_9"/>
   <xacro:x_tube_link name="right_arm4" child="motor5" extension="0.13315" twist="-3.7736" />
